File: eagle/rotor.sch (EAGLE design)
At the start: 53 parts, among them IC1 TXS0108, IC2 7815TV, J1 PL9823, J2 pwr2, J3 Power, J4 Antenna, J5 Power, J6 CCW, J7 Brake, J8 CW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

Commit message: eagle
Parts:
- J4: device TB004-508-02BE:TB004-508-02BE -> TB004-508-03BE:TB004-508-03BE
- Q1: device test:2N2907 -> test:2N2907CBE
- R3: value 1100 -> 1100 Ω
- T1: device test:2N2222 -> test:2N2222CBE
Connections:
- net +5V: now also Q1.C; no longer Q1.E
- net GND: now also J4.3
- net N$8: now also Q1.E; no longer Q1.C
Other:
- moved on the sheet: C1, C2, C3, IC2, Q1, R18, R3, U3G2, U3G3

Commit message: add dpdt switch
Parts:
- added J10: TB004-508-02BE, TB004-508-02BE:TB004-508-02BE
- added TEST-SW: DPDT-SWITCH, ladyada:DPDT-SWITCH
- R3: device test:R-US_0204/7 -> ladyada:R-US_M0805
Connections:
- new net N$13: R3.1, TEST-SW.C-1, TEST-SW.C-2
- new net N$14: J10.2, TEST-SW.NC-1, TEST-SW.NC-2
- net GND: now also J10.1
- net ROOF-3: now also TEST-SW.NO-1, TEST-SW.NO-2; no longer R2.1, R3.1
Changed lines of the file:
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@@
 <part name="R2" library="test" deviceset="R-US_" device="M0805" package3d_urn="urn:adsk.eagle:package:6240587/1" value="100k"/>
 <part name="D1" library="diode" library_urn="urn:adsk.eagle:library:210" deviceset="ZENER-DIODE" device="ZD-7.5" package3d_urn="urn:adsk.eagle:package:43411/1" value="5.1v 2%"/>
-<part name="R3" library="test" deviceset="R-US_" device="0204/7" package3d_urn="urn:adsk.eagle:package:6240596/1" value="1100 Ω"/>
+<part name="R3" library="ladyada" deviceset="R-US_" device="M0805" package3d_urn="urn:adsk.eagle:package:6240587/1" value="1100 Ω"/>
 <part name="R4" library="test" deviceset="R-US_" device="M0805" package3d_urn="urn:adsk.eagle:package:6240587/1" value="1k"/>
 <part name="R5" library="test" deviceset="R-US_" device="M0805" package3d_urn="urn:adsk.eagle:package:6240587/1" value="1k"/>
@@
 <part name="J4" library="TB004-508-03BE" deviceset="TB004-508-03BE" device="" value="Antenna"/>
 <part name="SUPPLY4" library="Power_Symbols" library_urn="urn:adsk.eagle:library:16502351" deviceset="EGND" device="" value="GND"/>
+<part name="TEST-SW" library="ladyada" deviceset="DPDT-SWITCH" device=""/>
+<part name="J10" library="TB004-508-02BE" deviceset="TB004-508-02BE" device=""/>
+<part name="SUPPLY6" library="Power_Symbols" library_urn="urn:adsk.eagle:library:16502351" deviceset="EGND" device="" value="GND"/>
 </parts>
 <sheets>
@@
 <attribute name="VALUE" x="-219.71" y="82.042" size="1.778" layer="96" rot="R180"/>
 </instance>
-<instance part="SUPPLY3" gate="G$1" x="-208.28" y="15.24" smashed="yes">
-<attribute name="VALUE" x="-208.407" y="11.303" size="1.778" layer="96" align="bottom-center"/>
+<instance part="SUPPLY3" gate="G$1" x="-208.28" y="12.7" smashed="yes">
+<attribute name="VALUE" x="-208.407" y="8.763" size="1.778" layer="96" align="bottom-center"/>
 </instance>
 <instance part="J4" gate="G$1" x="-218.44" y="127" smashed="yes" rot="R90">
@@
 <instance part="SUPPLY4" gate="G$1" x="-205.74" y="104.14" smashed="yes">
 <attribute name="VALUE" x="-205.867" y="100.203" size="1.778" layer="96" align="bottom-center"/>
+</instance>
+<instance part="TEST-SW" gate="G$1" x="-284.48" y="109.22" smashed="yes">
+<attribute name="NAME" x="-294.132" y="104.14" size="1.778" layer="95" rot="R90"/>
+<attribute name="VALUE" x="-273.05" y="104.14" size="1.778" layer="96" rot="R90"/>
+</instance>
+<instance part="J10" gate="G$1" x="-320.04" y="119.38" smashed="yes" rot="R180">
+<attribute name="NAME" x="-314.46" y="114.3" size="1.778" layer="95" rot="R180"/>
+<attribute name="VALUE" x="-314.96" y="124.46" size="1.778" layer="96" rot="R180"/>
+</instance>
+<instance part="SUPPLY6" gate="G$1" x="-304.8" y="53.34" smashed="yes">
+<attribute name="VALUE" x="-304.927" y="49.403" size="1.778" layer="96" align="bottom-center"/>
 </instance>
 </instances>
@@
 <net name="GND" class="0">
 <segment>
+<pinref part="SUPPLY6" gate="G$1" pin="EGND"/>
+<wire x1="-304.8" y1="55.88" x2="-304.8" y2="60.96" width="0.1524" layer="91"/>
 <wire x1="-68.58" y1="0" x2="-68.58" y2="7.62" width="0.1524" layer="91"/>
 <wire x1="-68.58" y1="7.62" x2="-68.58" y2="33.02" width="0.1524" layer="91"/>
@@
 <wire x1="-35.56" y1="7.62" x2="-58.42" y2="7.62" width="0.1524" layer="91"/>
 <wire x1="-58.42" y1="7.62" x2="-68.58" y2="7.62" width="0.1524" layer="91"/>
-<wire x1="-165.1" y1="27.94" x2="-165.1" y2="22.86" width="0.1524" layer="91"/>
-<wire x1="-165.1" y1="22.86" x2="-104.14" y2="22.86" width="0.1524" layer="91"/>
-<wire x1="-104.14" y1="22.86" x2="-104.14" y2="33.02" width="0.1524" layer="91"/>
+<wire x1="-165.1" y1="27.94" x2="-165.1" y2="20.32" width="0.1524" layer="91"/>
+<wire x1="-165.1" y1="20.32" x2="-104.14" y2="20.32" width="0.1524" layer="91"/>
+<wire x1="-104.14" y1="20.32" x2="-104.14" y2="33.02" width="0.1524" layer="91"/>
 <junction x="-104.14" y="33.02"/>
 <pinref part="R4" gate="G$1" pin="1"/>
-<wire x1="-172.72" y1="25.4" x2="-172.72" y2="22.86" width="0.1524" layer="91"/>
-<wire x1="-172.72" y1="22.86" x2="-165.1" y2="22.86" width="0.1524" layer="91"/>
-<junction x="-165.1" y="22.86"/>
+<wire x1="-172.72" y1="25.4" x2="-172.72" y2="20.32" width="0.1524" layer="91"/>
+<wire x1="-172.72" y1="20.32" x2="-165.1" y2="20.32" width="0.1524" layer="91"/>
+<junction x="-165.1" y="20.32"/>
 <pinref part="R5" gate="G$1" pin="1"/>
-<wire x1="-180.34" y1="25.4" x2="-180.34" y2="22.86" width="0.1524" layer="91"/>
-<wire x1="-180.34" y1="22.86" x2="-172.72" y2="22.86" width="0.1524" layer="91"/>
-<junction x="-172.72" y="22.86"/>
+<wire x1="-180.34" y1="25.4" x2="-180.34" y2="20.32" width="0.1524" layer="91"/>
+<wire x1="-180.34" y1="20.32" x2="-172.72" y2="20.32" width="0.1524" layer="91"/>
+<junction x="-172.72" y="20.32"/>
 <pinref part="C6" gate="G$1" pin="2"/>
 <wire x1="-58.42" y1="25.4" x2="-58.42" y2="7.62" width="0.1524" layer="91"/>
@@
 <pinref part="SUPPLY5" gate="G$1" pin="EGND"/>
 <wire x1="-78.74" y1="106.68" x2="-78.74" y2="109.22" width="0.1524" layer="91"/>
-<wire x1="-180.34" y1="22.86" x2="-208.28" y2="22.86" width="0.1524" layer="91"/>
-<junction x="-180.34" y="22.86"/>
+<wire x1="-180.34" y1="20.32" x2="-208.28" y2="20.32" width="0.1524" layer="91"/>
+<junction x="-180.34" y="20.32"/>
 <pinref part="C10" gate="G$1" pin="2"/>
 <wire x1="-231.14" y1="63.5" x2="-231.14" y2="60.96" width="0.1524" layer="91"/>
@@
 <pinref part="T1" gate="G$1" pin="E"/>
 <wire x1="-208.28" y1="60.96" x2="-208.28" y2="73.66" width="0.1524" layer="91"/>
-<wire x1="-208.28" y1="22.86" x2="-208.28" y2="60.96" width="0.1524" layer="91"/>
+<wire x1="-208.28" y1="20.32" x2="-208.28" y2="60.96" width="0.1524" layer="91"/>
 <junction x="-208.28" y="60.96"/>
 <pinref part="SUPPLY3" gate="G$1" pin="EGND"/>
-<wire x1="-208.28" y1="17.78" x2="-208.28" y2="22.86" width="0.1524" layer="91"/>
-<junction x="-208.28" y="22.86"/>
+<wire x1="-208.28" y1="15.24" x2="-208.28" y2="20.32" width="0.1524" layer="91"/>
+<junction x="-208.28" y="20.32"/>
 <pinref part="J4" gate="G$1" pin="3"/>
 <wire x1="-215.9" y1="116.84" x2="-215.9" y2="109.22" width="0.1524" layer="91"/>
@@
 <wire x1="-205.74" y1="106.68" x2="-205.74" y2="109.22" width="0.1524" layer="91"/>
 <junction x="-205.74" y="109.22"/>
+<pinref part="J10" gate="G$1" pin="1"/>
+<wire x1="-309.88" y1="116.84" x2="-304.8" y2="116.84" width="0.1524" layer="91"/>
+<wire x1="-304.8" y1="116.84" x2="-304.8" y2="60.96" width="0.1524" layer="91"/>
+<wire x1="-304.8" y1="60.96" x2="-231.14" y2="60.96" width="0.1524" layer="91"/>
+<junction x="-231.14" y="60.96"/>
+<junction x="-304.8" y="60.96"/>
 </segment>
 </net>
@@
 <net name="ROOF-3" class="0">
 <segment>
-<pinref part="R2" gate="G$1" pin="1"/>
-<wire x1="-157.48" y1="111.76" x2="-157.48" y2="96.52" width="0.1524" layer="91"/>
-<wire x1="-220.98" y1="116.84" x2="-220.98" y2="96.52" width="0.1524" layer="91"/>
-<wire x1="-220.98" y1="96.52" x2="-157.48" y2="96.52" width="0.1524" layer="91"/>
-<pinref part="R3" gate="G$1" pin="1"/>
-<wire x1="-157.48" y1="96.52" x2="-17.78" y2="96.52" width="0.1524" layer="91"/>
-<wire x1="-17.78" y1="96.52" x2="-17.78" y2="124.46" width="0.1524" layer="91"/>
-<junction x="-157.48" y="96.52"/>
+<wire x1="-220.98" y1="116.84" x2="-220.98" y2="104.14" width="0.1524" layer="91"/>
 <label x="-45.72" y="96.52" size="1.778" layer="95"/>
 <label x="-180.34" y="96.52" size="1.778" layer="95"/>
 <pinref part="J4" gate="G$1" pin="1"/>
 <label x="-220.98" y="106.68" size="1.778" layer="95" rot="R90"/>
+<wire x1="-220.98" y1="104.14" x2="-259.08" y2="104.14" width="0.1524" layer="91"/>
+<wire x1="-259.08" y1="104.14" x2="-259.08" y2="127" width="0.1524" layer="91"/>
+<wire x1="-259.08" y1="127" x2="-281.94" y2="127" width="0.1524" layer="91"/>
+<pinref part="TEST-SW" gate="G$1" pin="NO-1"/>
+<wire x1="-287.02" y1="114.3" x2="-287.02" y2="121.92" width="0.1524" layer="91"/>
+<wire x1="-287.02" y1="121.92" x2="-281.94" y2="121.92" width="0.1524" layer="91"/>
+<pinref part="TEST-SW" gate="G$1" pin="NO-2"/>
+<wire x1="-281.94" y1="121.92" x2="-276.86" y2="121.92" width="0.1524" layer="91"/>
+<wire x1="-276.86" y1="121.92" x2="-276.86" y2="114.3" width="0.1524" layer="91"/>
+<wire x1="-281.94" y1="127" x2="-281.94" y2="121.92" width="0.1524" layer="91"/>
+<junction x="-281.94" y="121.92"/>
 </segment>
 </net>
@@
 </segment>
 </net>
+<net name="N$13" class="0">
+<segment>
+<pinref part="TEST-SW" gate="G$1" pin="C-1"/>
+<pinref part="TEST-SW" gate="G$1" pin="C-2"/>
+<wire x1="-289.56" y1="104.14" x2="-284.48" y2="104.14" width="0.1524" layer="91"/>
+<wire x1="-284.48" y1="104.14" x2="-279.4" y2="104.14" width="0.1524" layer="91"/>
+<wire x1="-284.48" y1="104.14" x2="-284.48" y2="96.52" width="0.1524" layer="91"/>
+<wire x1="-284.48" y1="96.52" x2="-17.78" y2="96.52" width="0.1524" layer="91"/>
+<junction x="-284.48" y="104.14"/>
+<pinref part="R3" gate="G$1" pin="1"/>
+<wire x1="-17.78" y1="96.52" x2="-17.78" y2="124.46" width="0.1524" layer="91"/>
+</segment>
+</net>
+<net name="N$14" class="0">
+<segment>
+<pinref part="TEST-SW" gate="G$1" pin="NC-1"/>
+<wire x1="-292.1" y1="114.3" x2="-292.1" y2="119.38" width="0.1524" layer="91"/>
+<wire x1="-292.1" y1="119.38" x2="-281.94" y2="119.38" width="0.1524" layer="91"/>
+<pinref part="TEST-SW" gate="G$1" pin="NC-2"/>
+<wire x1="-281.94" y1="119.38" x2="-281.94" y2="114.3" width="0.1524" layer="91"/>
+<pinref part="J10" gate="G$1" pin="2"/>
+<wire x1="-309.88" y1="119.38" x2="-292.1" y2="119.38" width="0.1524" layer="91"/>
+<junction x="-292.1" y="119.38"/>
+</segment>
+</net>
